File: 555_chaser.kicad_pcb (KiCad board)
At the start: 2 copper layers, 42.9 x 73.8 mm, 19 parts, among them J1 Conn_01x02_Socket, J2 Conn_01x01_Socket, U1 NE555P, U3 4017

Commit message: Add files via upload
deleted J2 and made the J1 a 3 block terminal; width 3.5mm
Parts:
- removed J2: Conn_01x01_Socket, Connector_PinHeader_2.54mm:PinHeader_1x01_P2.54mm_Vertical
- J1: value Conn_01x02_Socket -> Conn_01x03_Socket; footprint Connector_PinHeader_2.54mm:PinHeader_1x02_P2.54mm_Vertical -> TerminalBlock_4Ucon:TerminalBlock_4Ucon_1x03_P3.50mm_Horizontal
- moved J1 4.54 mm to (210.5, 123.5), turned to 90 degrees
Routing:
- net OUT: track 32.1 -> 51.6 mm
- net Net-(D4-A): track 34.9 -> 32.1 mm
- net GND: track 102.5 -> 103.8 mm
